File: MikeRoberts.sch (KiCad schematic (older format))
At the start: 6 parts, among them U1 LM321

Commit message: Final push
Updated schematics + layout files
Parts:
- added J1, J2: CONN_01X02_MALE, Measurement_Points:Test_Point_2Pads, symbol CONN_01X02_MALE
- C1, R2: footprint (none) -> Resistors_THT:R_Axial_DIN0204_L3.6mm_D1.6mm_P5.08mm_Horizontal
- D1: footprint Thru-Hole -> Resistors_THT:R_Axial_DIN0204_L3.6mm_D1.6mm_P5.08mm_Horizontal
- RV1, RV2: footprint (none) -> Potentiometers:Potentiometer_Trimmer_Vishay_T73YP_Horizontal
- U1: footprint (none) -> TO_SOT_Packages_SMD:SOT-23-5_HandSoldering; symbol LM7332 -> LM321
Connections:
- net labels added: VIN, VOUT
- wire segments 17 -> 22
Other:
- note added: "J1 and J2 can be populated with standard 2.54mm pitch headers. For the sake of this exercise, we will solder wires to avoid additional BOM components."
- moved on the sheet: D1
Changed lines of the file:
@@
 LIBS:contrib
 LIBS:valves
+LIBS:MikeRoberts-cache
 EELAYER 25 0
 EELAYER END
@@
 L D_Zener D1
 U 1 1 58DB138D
-P 4200 3800
-F 0 "D1" H 4200 3900 50  0000 C CNN
-F 1 "2.1V" H 4200 3700 50  0000 C CNN
-F 2 "Thru-Hole" H 4200 3800 50  0001 C CNN
-F 3 "" H 4200 3800 50  0001 C CNN
-F 4 "Nexperia" H 4200 3800 60  0001 C CNN "MFR"
-F 5 "NZX2V1B,133" H 4200 3800 60  0001 C CNN "MFG PN"
-F 6 "1727-1134-1-ND" H 4200 3800 60  0001 C CNN "Vendor PN"
-F 7 "Digi-Key" H 4200 3800 60  0001 C CNN "Vendor"
-	1    4200 3800
+P 4200 3850
+F 0 "D1" H 4200 3950 50  0000 C CNN
+F 1 "2.1V" H 4200 3750 50  0000 C CNN
+F 2 "Resistors_THT:R_Axial_DIN0204_L3.6mm_D1.6mm_P5.08mm_Horizontal" H 4200 3850 50  0001 C CNN
+F 3 "" H 4200 3850 50  0001 C CNN
+F 4 "Nexperia" H 4200 3850 60  0001 C CNN "MFR"
+F 5 "NZX2V1B,133" H 4200 3850 60  0001 C CNN "MFG PN"
+F 6 "1727-1134-1-ND" H 4200 3850 60  0001 C CNN "Vendor PN"
+F 7 "Digi-Key" H 4200 3850 60  0001 C CNN "Vendor"
+	1    4200 3850
 	0    -1   1    0
 $EndComp
@@
 L GND #PWR01
 U 1 1 58DB1510
-P 4200 3950
-F 0 "#PWR01" H 4200 3700 50  0001 C CNN
-F 1 "GND" H 4200 3800 50  0000 C CNN
-F 2 "" H 4200 3950 50  0001 C CNN
-F 3 "" H 4200 3950 50  0001 C CNN
-	1    4200 3950
+P 4200 4050
+F 0 "#PWR01" H 4200 3800 50  0001 C CNN
+F 1 "GND" H 4200 3900 50  0000 C CNN
+F 2 "" H 4200 4050 50  0001 C CNN
+F 3 "" H 4200 4050 50  0001 C CNN
+	1    4200 4050
 	1    0    0    -1
 $EndComp
@@
 F 0 "RV1" V 4675 3650 50  0000 C CNN
 F 1 "POT" V 4750 3650 50  0000 C CNN
-F 2 "" H 4850 3650 50  0001 C CNN
+F 2 "Potentiometers:Potentiometer_Trimmer_Vishay_T73YP_Horizontal" H 4850 3650 50  0001 C CNN
 F 3 "" H 4850 3650 50  0001 C CNN
 	1    4850 3650
@@
 F 0 "R2" V 6580 4650 50  0000 C CNN
 F 1 "15k" V 6500 4650 50  0000 C CNN
-F 2 "" V 6430 4650 50  0001 C CNN
+F 2 "Resistors_THT:R_Axial_DIN0204_L3.6mm_D1.6mm_P5.08mm_Horizontal" V 6430 4650 50  0001 C CNN
 F 3 "" H 6500 4650 50  0001 C CNN
 	1    6500 4650
@@
 F 0 "RV2" V 5675 4100 50  0000 C CNN
 F 1 "POT" V 5750 4100 50  0000 C CNN
-F 2 "" H 5850 4100 50  0001 C CNN
+F 2 "Potentiometers:Potentiometer_Trimmer_Vishay_T73YP_Horizontal" H 5850 4100 50  0001 C CNN
 F 3 "" H 5850 4100 50  0001 C CNN
 	1    5850 4100
@@
 F 0 "C1" H 5425 4000 50  0000 L CNN
 F 1 "0.1uF" H 5425 3800 50  0000 L CNN
-F 2 "" H 5438 3750 50  0001 C CNN
+F 2 "Resistors_THT:R_Axial_DIN0204_L3.6mm_D1.6mm_P5.08mm_Horizontal" H 5438 3750 50  0001 C CNN
 F 3 "" H 5400 3900 50  0001 C CNN
 	1    5400 3900
@@
 	5400 4050 5400 4300
 $Comp
-L GND #PWR?
+L GND #PWR06
 U 1 1 58DB3D89
 P 5400 4300
-F 0 "#PWR?" H 5400 4050 50  0001 C CNN
+F 0 "#PWR06" H 5400 4050 50  0001 C CNN
 F 1 "GND" H 5400 4150 50  0000 C CNN
 F 2 "" H 5400 4300 50  0001 C CNN
@@
 $EndComp
 $Comp
-L LM7332 U1
+L LM321 U1
 U 1 1 58DB161C
 P 6250 3750
 F 0 "U1" H 6250 3900 50  0000 L CNN
 F 1 "LM321" H 6250 3600 50  0000 L CNN
-F 2 "" H 6150 3800 50  0001 C CNN
+F 2 "TO_SOT_Packages_SMD:SOT-23-5_HandSoldering" H 6150 3800 50  0001 C CNN
 F 3 "" H 6250 3900 50  0001 C CNN
 	1    6250 3750
@@
 Text Notes 8150 7650 0    60   ~ 0
 3/28/17
+$Comp
+L CONN_01X02_MALE J1
+U 1 1 58DB6987
+P 3450 4100
+F 0 "J1" H 3450 4275 50  0000 C CNN
+F 1 "CONN_01X02_MALE" H 3450 3900 50  0000 C CNN
+F 2 "Measurement_Points:Test_Point_2Pads" H 3450 4200 50  0001 C CNN
+F 3 "" H 3450 4200 50  0001 C CNN
+	1    3450 4100
+	1    0    0    -1
+$EndComp
+$Comp
+L CONN_01X02_MALE J2
+U 1 1 58DB69C8
+P 7550 4100
+F 0 "J2" H 7550 4275 50  0000 C CNN
+F 1 "CONN_01X02_MALE" H 7550 3900 50  0000 C CNN
+F 2 "Measurement_Points:Test_Point_2Pads" H 7550 4200 50  0001 C CNN
+F 3 "" H 7550 4200 50  0001 C CNN
+	1    7550 4100
+	-1   0    0    1
+$EndComp
+$Comp
+L GND #PWR07
+U 1 1 58DB6A25
+P 3750 4200
+F 0 "#PWR07" H 3750 3950 50  0001 C CNN
+F 1 "GND" H 3750 4050 50  0000 C CNN
+F 2 "" H 3750 4200 50  0001 C CNN
+F 3 "" H 3750 4200 50  0001 C CNN
+	1    3750 4200
+	1    0    0    -1
+$EndComp
+$Comp
+L GND #PWR08
+U 1 1 58DB6A49
+P 7250 4200
+F 0 "#PWR08" H 7250 3950 50  0001 C CNN
+F 1 "GND" H 7250 4050 50  0000 C CNN
+F 2 "" H 7250 4200 50  0001 C CNN
+F 3 "" H 7250 4200 50  0001 C CNN
+	1    7250 4200
+	1    0    0    -1
+$EndComp
+Wire Wire Line
+	3750 4000 3950 4000
+Wire Wire Line
+	3950 4000 3950 3650
+Connection ~ 3950 3650
+Text Label 3800 4000 0    60   ~ 0
+VIN
+Wire Wire Line
+	6750 4000 7250 4000
+Connection ~ 6750 4000
+Text Label 7000 4000 0    60   ~ 0
+VOUT
+Text Notes 2550 5700 0    60   ~ 0
+J1 and J2 can be populated with standard 2.54mm pitch headers.  For the sake of this exercise, we will solder wires to avoid additional BOM components.
+Wire Wire Line
+	4200 3650 4200 3700
+Connection ~ 4200 3650
+Wire Wire Line
+	4200 4050 4200 4000
 $EndSCHEMATC
