File: Final Submission Files/MikeRoberts.kicad_pcb (KiCad board)
At the start: 2 copper layers, 45.7 x 43.2 mm, 8 parts, among them J1 CONN_01X02_MALE, J2 CONN_01X02_MALE, U1 LM321

Commit message: Final push
Updated schematics + layout files
Parts:
- J1: value CONN_01X02_MALE -> INPUT HEADER
- J2: value CONN_01X02_MALE -> OUTPUT HEADER
- moved D1 33.7 mm to (154.9, 85.1), turned to 0 degrees
Connections:
- D1 pad 1: Input -> Net-(D1-Pad1)
Routing:
- net Input: track 13.8 -> 8.15 mm
- net GND: track 75.8 -> 75.3 mm
